File: StackDriver/board.brd (EAGLE design)
At the start: 106.7 x 85.1 mm, 49 parts, among them IC1 LM741P, IC10 LM741P, IC11 LM741P, IC12 LM741P, IC13 LM741P, IC14 LM741P, IC15 LM741P, IC2 LM741P, IC3 LM741P, IC4 LM741P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

Commit message: Brzydko wyglądająca ścieżka przy wejściach: POPRAWIONA
Routing:
- net V-: track 415.7 -> 415.1 mm
Changed lines of the file:
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@@
 <layer number="17" name="Pads" color="2" fill="1" visible="yes" active="yes"/>
 <layer number="18" name="Vias" color="2" fill="1" visible="yes" active="yes"/>
-<layer number="19" name="Unrouted" color="6" fill="1" visible="no" active="yes"/>
+<layer number="19" name="Unrouted" color="6" fill="1" visible="yes" active="yes"/>
 <layer number="20" name="Dimension" color="24" fill="1" visible="no" active="yes"/>
 <layer number="21" name="tPlace" color="7" fill="1" visible="no" active="yes"/>
@@
 <wire x1="35.56" y1="25.4" x2="35.56" y2="27.94" width="0.5" layer="1"/>
 <wire x1="35.56" y1="27.94" x2="36.83" y2="29.21" width="0.5" layer="1"/>
-<wire x1="85.09" y1="7.62" x2="85.09" y2="8.89" width="0.5" layer="1"/>
-<wire x1="86.068" y1="7.48099375" x2="86.068" y2="7.912" width="0.5" layer="1"/>
-<wire x1="86.068" y1="7.912" x2="85.09" y2="8.89" width="0.5" layer="1"/>
-<wire x1="103.41" y1="8.785225" x2="97.604775" y2="2.98" width="0.5" layer="1"/>
-<wire x1="97.604775" y1="2.98" x2="90.56899375" y2="2.98" width="0.5" layer="1"/>
-<wire x1="90.56899375" y1="2.98" x2="86.068" y2="7.48099375" width="0.5" layer="1"/>
+<wire x1="97.604775" y1="2.98" x2="103.41" y2="8.785225" width="0.5" layer="1"/>
 <wire x1="103.41" y1="49.53" x2="103.41" y2="26.67" width="0.5" layer="1"/>
 <wire x1="103.41" y1="26.67" x2="103.41" y2="8.785225" width="0.5" layer="1"/>
@@
 <wire x1="100.69" y1="23.95" x2="103.41" y2="26.67" width="0.5" layer="1"/>
 <wire x1="97.97" y1="23.95" x2="100.69" y2="23.95" width="0.5" layer="1"/>
+<wire x1="85.09" y1="8.84" x2="85.09" y2="8.6662" width="0.1524" layer="1"/>
+<wire x1="85.09" y1="8.89" x2="85.09" y2="8.84" width="0.5" layer="1"/>
+<wire x1="85.09" y1="8.89" x2="85.09" y2="7.62" width="0.5" layer="1"/>
+<wire x1="85.09" y1="7.62" x2="89.73" y2="2.98" width="0.5" layer="1"/>
+<wire x1="89.73" y1="2.98" x2="97.604775" y2="2.98" width="0.5" layer="1"/>
 </signal>
 <signal name="15">

Commit message: debug
Routing:
- net GND: track 537.5 -> 519.7 mm
